Commit message: removed deprecated files and re-built

File: go2/go2_description/xacro/leg.xacro (robot description, xacro)
@@ -57,5 +57,5 @@
                 </xacro:if>
                 <geometry>
-                    <mesh filename="file://$(find go2_description)/meshes/hip.dae" scale="1 1 1"/>
+                    <mesh filename="file://$(find go2_description)/dae/hip.dae" scale="1 1 1"/>
                 </geometry>
                 <!-- <material name="orange"/> -->
@@ -117,8 +117,8 @@
                 <geometry>
                     <xacro:if value="${mirror_dae == True}">
-                        <mesh filename="file://$(find go2_description)/meshes/thigh.dae" scale="1 1 1"/>
+                        <mesh filename="file://$(find go2_description)/dae/thigh.dae" scale="1 1 1"/>
                     </xacro:if>
                     <xacro:if value="${mirror_dae == False}">
-                        <mesh filename="file://$(find go2_description)/meshes/thigh_mirror.dae" scale="1 1 1"/>
+                        <mesh filename="file://$(find go2_description)/dae/thigh_mirror.dae" scale="1 1 1"/>
                     </xacro:if>
                 </geometry>
@@ -182,5 +182,5 @@
                 <origin rpy="0 0 0" xyz="0 0 0"/>
                 <geometry>
-                    <mesh filename="file://$(find go2_description)/meshes/calf.dae" scale="1 1 1"/>
+                    <mesh filename="file://$(find go2_description)/dae/calf.dae" scale="1 1 1"/>
                 </geometry>
                 <!-- <material name="orange"/> -->

File: go2/go2_description/xacro/robot.xacro (robot description, xacro)
@@ -33,5 +33,5 @@
             <origin rpy="0 0 0" xyz="0 0 0"/>
             <geometry>
-                <mesh filename="file://$(find go2_description)/meshes/trunk.dae" scale="1 1 1"/>
+                <mesh filename="file://$(find go2_description)/dae/base.dae" scale="1 1 1"/>
             </geometry>
             <!-- <material name="orange"/> -->

File: go2/go2_description/xacro/robot_camera.xacro (robot description, xacro)
@@ -33,5 +33,5 @@
             <origin rpy="0 0 0" xyz="0 0 0"/>
             <geometry>
-                <mesh filename="file://$(find go2_description)/meshes/trunk.dae" scale="1 1 1"/>
+                <mesh filename="file://$(find go2_description)/dae/base.dae" scale="1 1 1"/>
             </geometry>
             <!-- <material name="orange"/> -->
